Commit message: middle change

File: MATLAB/haoran_model/Arm_version_1.0/robots/V1_Arm_URDF.URDF (robot description, URDF)
Before this commit: robot V1_Arm_URDF, 18 links, 17 joints
Links:
- link V1_arm1_tool_translate_link: mass 0.800 -> 0.950
Joints:
- joint V1_arm1_tool_rotate_joint: origin xyz=0 0 -0.1891 rpy=0 0 0 -> xyz=0 0 0 rpy=0 0 0
- joint V1_arm1_wrist_joint: origin xyz=0 0 0 rpy=1.5708 1.5708 0 -> xyz=0 0 -0.1891 rpy=1.5708 1.5708 0
