Commit message: Resolve the conflict between bed_adapter_review and master

File: MATLAB/haoran_model/2015_drawer_urdf_3a/robots/2015_drawer_urdf_3a.URDF (robot description, URDF)
Before this commit: robot 2015_drawer_urdf_3a, 4 links, 3 joints
Joints:
- joint dummy_link: origin xyz=-0.18149 0.0063436 0.083002 rpy=0 0 3.1415 -> xyz=-0.192576 0.0063436 0.11251 rpy=0 0 1.571

Commit message: 1. Update dummy link in table adapter URDF for new base transform 2.  Update .mat files for table adapter for new base transform
 MATLAB/haoran_model/data/bed_adapter_info.mat
	modified:   MATLAB/haoran_model/data/vertex_bed.mat

1.  Update dummy link in table adapter URDF for new base transform
2.  Update .mat files for table adapter for new base transform

Change-Id: Iff6399463eac04e396644f8be01ef576bb6a9b94

File: MATLAB/haoran_model/2015_drawer_urdf_3a/robots/2015_drawer_urdf_3a.URDF (robot description, URDF)
Before this commit: robot 2015_drawer_urdf_3a, 4 links, 3 joints
Joints:
- joint dummy_link: origin xyz=-0.192576 0.0063436 0.11251 rpy=0 0 1.571 -> xyz=-0.192576 0.0063436 0.11251 rpy=1.571 0 0

File: MATLAB/haoran_model/2015_drawer_urdf_3a/robots/drawers.urdf (robot description, URDF)
Before this commit: robot drawers, 50 links, 49 joints
Joints:
- joint drawer0_dummy_joint: origin xyz=-0.192576 0.0063436 0.11251 rpy=0 0 1.571 -> xyz=-0.192576 0.0063436 0.11251 rpy=1.571 0 0
- joint drawer1_dummy_joint: origin xyz=-0.192576 0.0063436 0.11251 rpy=0 0 1.571 -> xyz=-0.192576 0.0063436 0.11251 rpy=1.571 0 0
- joint drawer2_dummy_joint: origin xyz=-0.192576 0.0063436 0.11251 rpy=0 0 1.571 -> xyz=-0.192576 0.0063436 0.11251 rpy=1.571 0 0
- joint drawer3_dummy_joint: origin xyz=-0.192576 0.0063436 0.11251 rpy=0 0 1.571 -> xyz=-0.192576 0.0063436 0.11251 rpy=1.571 0 0
- joint drawer4_dummy_joint: origin xyz=-0.192576 0.0063436 0.11251 rpy=0 0 1.571 -> xyz=-0.192576 0.0063436 0.11251 rpy=1.571 0 0
- joint drawer5_dummy_joint: origin xyz=-0.192576 0.0063436 0.11251 rpy=0 0 1.571 -> xyz=-0.192576 0.0063436 0.11251 rpy=1.571 0 0
- joint drawer6_dummy_joint: origin xyz=-0.192576 0.0063436 0.11251 rpy=0 0 1.571 -> xyz=-0.192576 0.0063436 0.11251 rpy=1.571 0 0
- joint drawer7_dummy_joint: origin xyz=-0.192576 0.0063436 0.11251 rpy=0 0 1.571 -> xyz=-0.192576 0.0063436 0.11251 rpy=1.571 0 0
